Commit message: pick_sponge_and_add_the_ability_hand

File: assets/robot/ability_hand_description/ability_hand_right.urdf (robot description, URDF)
Before this commit: robot ability_hand, 17 links, 16 joints
Links:
- removed link base
- added link base_link, mass 0.200; visual mesh filename=models/wristmesh.STL
Joints:
- joint wrist2thumb: parent base -> base_link

File: assets/robot/xarm6_description/xarm6_ability_left.urdf (robot description, URDF)
Before this commit: robot xarm6, 30 links, 29 joints
Links:
- removed link link_0.0
- removed link link_1.0
- removed link link_10.0
- removed link link_11.0
- removed link link_11.0_tip
- removed link link_12.0
- removed link link_13.0
- removed link link_14.0
- removed link link_15.0
- removed link link_15.0_tip
- removed link link_2.0
- removed link link_3.0
- removed link link_3.0_tip
- removed link link_4.0
- removed link link_5.0
- removed link link_6.0
- removed link link_7.0
- removed link link_7.0_tip
- removed link link_8.0
- removed link link_9.0
- removed link palm
- removed link wrist
- added link index_L1, mass 0.00635888; visual mesh filename=models/idx-F1.STL
- added link index_L2, mass 0.00645; visual mesh filename=models/idx-F2.STL
- added link index_anchor
- added link middle_L1, mass 0.00635888; visual mesh filename=models/idx-F1.STL
- added link middle_L2, mass 0.00645; visual mesh filename=models/idx-F2.STL
- added link middle_anchor
- added link pinky_L1, mass 0.00635888; visual mesh filename=models/idx-F1.STL
- added link pinky_L2, mass 0.00645; visual mesh filename=models/idx-F2.STL
- added link pinky_anchor
- added link ring_L1, mass 0.00635888; visual mesh filename=models/idx-F1.STL
- added link ring_L2, mass 0.00645; visual mesh filename=models/idx-F2.STL
- added link ring_anchor
- added link thumb_L1, mass 0.00268342; visual mesh filename=models/thumb-F1.STL
- added link thumb_L2, mass 0.0055; visual mesh filename=models/thumb-F2.STL
- added link thumb_anchor
- added link thumb_base, mass 0.400; visual mesh filename=models/FB_palm_ref.STL
- link base_link: mass 0.4154 -> 0.200; geometry visual mesh filename=models/wristmesh.STL
Joints:
- removed joint joint_0.0
- removed joint joint_1.0
- removed joint joint_10.0
- removed joint joint_11.0
- removed joint joint_11.0_tip
- removed joint joint_12.0
- removed joint joint_13.0
- removed joint joint_14.0
- removed joint joint_15.0
- removed joint joint_15.0_tip
- removed joint joint_2.0
- removed joint joint_3.0
- removed joint joint_3.0_tip
- removed joint joint_4.0
- removed joint joint_5.0
- removed joint joint_6.0
- removed joint joint_7.0
- removed joint joint_7.0_tip
- removed joint joint_8.0
- removed joint joint_9.0
- removed joint palm_joint
- removed joint wrist_joint
- added joint idx_anchor: type fixed, parent index_L2, child index_anchor, origin xyz=31.5541e-3  -10.44e-3 0.14e-3 rpy=0 0 0
- added joint index_q1: type revolute, parent thumb_base, child index_L1, origin xyz=-9.49e-3 -13.04e-3 -62.95e-3 rpy=-1.982050 1.284473 -2.090591, axis 0 0 1, limit lower=0 upper=2.0943951 effort=6.0 velocity=8.0677777442
- added joint index_q2: type revolute, parent index_L1, child index_L2, origin xyz=38.472723e-3 3.257695e-3 0.000000e-3 rpy=0 0 0.084474, axis 0 0 1, limit lower=0.0 upper=2.6586 effort=6.0 velocity=8.0677777442, mimic joint=index_q1 multiplier=1.05851325 offset=0.72349796
- added joint mid_anchor: type fixed, parent middle_L2, child middle_anchor, origin xyz=31.5541e-3  -10.44e-3 0.14e-3 rpy=0 0 0
- added joint middle_q1: type revolute, parent thumb_base, child middle_L1, origin xyz=9.653191e-3 -15.310271e-3 -67.853949e-3 rpy=-1.860531 1.308458 -1.896217, axis 0 0 1, limit lower=0 upper=2.0943951 effort=6.0 velocity=8.0677777442
- added joint middle_q2: type revolute, parent middle_L1, child middle_L2, origin xyz=38.472723e-3 3.257695e-3 0.000000 rpy=0 0 0.084474, axis 0 0 1, limit lower=0.0 upper=2.6586 effort=6.0 velocity=8.0677777442, mimic joint=middle_q1 multiplier=1.05851325 offset=0.72349796
- added joint pinky_q1: type revolute, parent thumb_base, child pinky_L1, origin xyz=49.521293e-3 -11.004583e-3 -63.029065e-3 rpy=-1.765110 1.322220 -1.658383, axis 0 0 1, limit lower=0 upper=2.0943951 effort=6.0 velocity=8.0677777442
- added joint pinky_q2: type revolute, parent pinky_L1, child pinky_L2, origin xyz=38.472723e-3 3.257695e-3 0.000000 rpy=0 0 0.084474, axis 0 0 1, limit lower=0.0 upper=2.6586 effort=6.0 velocity=8.0677777442, mimic joint=pinky_q1 multiplier=1.05851325 offset=0.72349796
- added joint pnky_anchor: type fixed, parent pinky_L2, child pinky_anchor, origin xyz=31.5541e-3  -10.44e-3 0.14e-3 rpy=0 0 0
- added joint ring_q1: type revolute, parent thumb_base, child ring_L1, origin xyz=29.954260e-3 -14.212492e-3 -67.286105e-3 rpy=-1.716598 1.321452 -1.675862, axis 0 0 1, limit lower=0 upper=2.0943951 effort=6.0 velocity=8.0677777442
- added joint ring_q2: type revolute, parent ring_L1, child ring_L2, origin xyz=38.472723e-3 3.257695e-3 0.000000 rpy=0 0 0.084474, axis 0 0 1, limit lower=0.0 upper=2.6586 effort=6.0 velocity=8.0677777442, mimic joint=ring_q1 multiplier=1.05851325 offset=0.72349796
- added joint rng_anchor: type fixed, parent ring_L2, child ring_anchor, origin xyz=31.5541e-3  -10.44e-3 0.14e-3 rpy=0 0 0
- added joint thmb_anchor: type fixed, parent thumb_L2, child thumb_anchor, origin xyz=52.0012259e-3  28.0086971e-3 -.884835778e-3 rpy=0 0 0
- added joint thumb_q1: type revolute, parent thumb_base, child thumb_L1, origin xyz=0 0 0 rpy=0 0 3.330437, axis 0 0 1, limit lower=-2.0943951 upper=0 effort=1.2 velocity=40.338888721
- added joint thumb_q2: type revolute, parent thumb_L1, child thumb_L2, origin xyz=27.8283501e-3 0 -14.7507000e-3 rpy=4.450589592585541 0 0, axis 0 0 1, limit lower=0 upper=2.0943951 effort=6.0 velocity=8.0677777442
- added joint wrist2thumb: type fixed, parent base_link, child thumb_base, origin xyz=24.0476665e-3 3.78124745e-3 32.32964923e-3 rpy=3.14148426 0.08848813 3.14036612
- joint gripper_base_joint: origin xyz=0 0.045 0.045 rpy=0 -1.57 -1.57 -> xyz=0 0 0 rpy=0 0 3.14

File: assets/robot/xarm6_description/xarm6_ability_right.urdf (robot description, URDF)
Before this commit: robot xarm6, 30 links, 29 joints
Links:
- removed link link_0.0
- removed link link_1.0
- removed link link_10.0
- removed link link_11.0
- removed link link_11.0_tip
- removed link link_12.0
- removed link link_13.0
- removed link link_14.0
- removed link link_15.0
- removed link link_15.0_tip
- removed link link_2.0
- removed link link_3.0
- removed link link_3.0_tip
- removed link link_4.0
- removed link link_5.0
- removed link link_6.0
- removed link link_7.0
- removed link link_7.0_tip
- removed link link_8.0
- removed link link_9.0
- removed link palm
- removed link wrist
- added link index_L1, mass 0.00635888; visual mesh filename=models/idx-F1.STL
- added link index_L2, mass 0.00645; visual mesh filename=models/idx-F2.STL
- added link index_anchor
- added link middle_L1, mass 0.00635888; visual mesh filename=models/idx-F1.STL
- added link middle_L2, mass 0.00645; visual mesh filename=models/idx-F2.STL
- added link middle_anchor
- added link pinky_L1, mass 0.00635888; visual mesh filename=models/idx-F1.STL
- added link pinky_L2, mass 0.00645; visual mesh filename=models/idx-F2.STL
- added link pinky_anchor
- added link ring_L1, mass 0.00635888; visual mesh filename=models/idx-F1.STL
- added link ring_L2, mass 0.00645; visual mesh filename=models/idx-F2.STL
- added link ring_anchor
- added link thumb_L1, mass 0.00268342; visual mesh filename=models/thumb-F1-MIR.STL
- added link thumb_L2, mass 0.0055; visual mesh filename=models/thumb-F2.STL
- added link thumb_anchor
- added link thumb_base, mass 0.200; visual mesh filename=models/FB_palm_ref_MIR.STL
- link base_link: mass 0.4154 -> 0.200; geometry visual mesh filename=models/wristmesh.STL
Joints:
- removed joint joint_0.0
- removed joint joint_1.0
- removed joint joint_10.0
- removed joint joint_11.0
- removed joint joint_11.0_tip
- removed joint joint_12.0
- removed joint joint_13.0
- removed joint joint_14.0
- removed joint joint_15.0
- removed joint joint_15.0_tip
- removed joint joint_2.0
- removed joint joint_3.0
- removed joint joint_3.0_tip
- removed joint joint_4.0
- removed joint joint_5.0
- removed joint joint_6.0
- removed joint joint_7.0
- removed joint joint_7.0_tip
- removed joint joint_8.0
- removed joint joint_9.0
- removed joint palm_joint
- removed joint wrist_joint
- added joint idx_anchor: type fixed, parent index_L2, child index_anchor, origin xyz=31.5541e-3  -10.44e-3 0.14e-3 rpy=0 0 0
- added joint index_q1: type revolute, parent thumb_base, child index_L1, origin xyz= 9.49e-3 -13.04e-3 -62.95e-3  rpy= -1.1595426535897932 1.284473 -1.0510016535897932 , axis 0 0 1, limit lower=0 upper=2.0943951 effort=6.0 velocity=8.0677777442
- added joint index_q2: type revolute, parent index_L1, child index_L2, origin xyz=38.472723e-3 3.257695e-3 0.000000e-3 rpy=0 0 0.084474, axis 0 0 1, limit lower=0.0 upper=2.6586 effort=6.0 velocity=8.0677777442, mimic joint=index_q1 multiplier=1.05851325 offset=0.72349796
- added joint mid_anchor: type fixed, parent middle_L2, child middle_anchor, origin xyz=31.5541e-3  -10.44e-3 0.14e-3 rpy=0 0 0
- added joint middle_q1: type revolute, parent thumb_base, child middle_L1, origin xyz= -9.653191e-3 -15.310271e-3 -67.853949e-3  rpy= -1.2810616535897934 1.308458 -1.2453756535897933 , axis 0 0 1, limit lower=0 upper=2.0943951 effort=6.0 velocity=8.0677777442
- added joint middle_q2: type revolute, parent middle_L1, child middle_L2, origin xyz=38.472723e-3 3.257695e-3 0.000000 rpy=0 0 0.084474, axis 0 0 1, limit lower=0.0 upper=2.6586 effort=6.0 velocity=8.0677777442, mimic joint=middle_q1 multiplier=1.05851325 offset=0.72349796
- added joint pinky_q1: type revolute, parent thumb_base, child pinky_L1, origin xyz= -49.521293e-3 -11.004583e-3 -63.029065e-3  rpy= -1.3764826535897934 1.32222 -1.4832096535897932 , axis 0 0 1, limit lower=0 upper=2.0943951 effort=6.0 velocity=8.0677777442
- added joint pinky_q2: type revolute, parent pinky_L1, child pinky_L2, origin xyz=38.472723e-3 3.257695e-3 0.000000 rpy=0 0 0.084474, axis 0 0 1, limit lower=0.0 upper=2.6586 effort=6.0 velocity=8.0677777442, mimic joint=pinky_q1 multiplier=1.05851325 offset=0.72349796
- added joint pnky_anchor: type fixed, parent pinky_L2, child pinky_anchor, origin xyz=31.5541e-3  -10.44e-3 0.14e-3 rpy=0 0 0
- added joint ring_q1: type revolute, parent thumb_base, child ring_L1, origin xyz= -29.95426e-3 -14.212492e-3 -67.286105e-3  rpy= -1.424994653589793 1.321452 -1.4657306535897934 , axis 0 0 1, limit lower=0 upper=2.0943951 effort=6.0 velocity=8.0677777442
- added joint ring_q2: type revolute, parent ring_L1, child ring_L2, origin xyz=38.472723e-3 3.257695e-3 0.000000 rpy=0 0 0.084474, axis 0 0 1, limit lower=0.0 upper=2.6586 effort=6.0 velocity=8.0677777442, mimic joint=ring_q1 multiplier=1.05851325 offset=0.72349796
- added joint rng_anchor: type fixed, parent ring_L2, child ring_anchor, origin xyz=31.5541e-3  -10.44e-3 0.14e-3 rpy=0 0 0
- added joint thmb_anchor: type fixed, parent thumb_L2, child thumb_anchor, origin xyz=52.00122724e-3 28.00869333e-3 6.98483578e-3 rpy=0 0 0
- added joint thumb_q1: type revolute, parent thumb_base, child thumb_L1, origin xyz= 0.0 0.0 0.0  rpy= 3.141592653589793 -0.0 -0.18884434641020664 , axis 0 0 1, limit lower=-2.0943951 upper=0 effort=1.2 velocity=40.338888721
- added joint thumb_q2: type revolute, parent thumb_L1, child thumb_L2, origin xyz= 27.8283501e-3 1.7436510745838653e-19 14.7507e-3  rpy= 1.832595714594045 -0.0 5.366520605522463e-18 , axis 0 0 1, limit lower=0 upper=2.0943951 effort=6.0 velocity=8.0677777442
- added joint wrist2thumb: type fixed, parent base_link, child thumb_base, origin xyz=-24.0476665e-3 3.78124745e-3 32.32964923e-3 rpy=3.14148426 -0.08848813 -3.14036612
- joint gripper_base_joint: origin xyz=0 0.045 0.045 rpy=0 -1.57 -1.57 -> xyz=0 0 0 rpy=0 0 3.14

File: assets/robot/xarm7_description/xarm7_ability_left.urdf (robot description, URDF)
Before this commit: robot xarm7, 32 links, 31 joints
Links:
- removed link link_0.0
- removed link link_1.0
- removed link link_10.0
- removed link link_11.0
- removed link link_11.0_tip
- removed link link_12.0
- removed link link_13.0
- removed link link_14.0
- removed link link_15.0
- removed link link_15.0_tip
- removed link link_2.0
- removed link link_3.0
- removed link link_3.0_tip
- removed link link_4.0
- removed link link_5.0
- removed link link_6.0
- removed link link_7.0
- removed link link_7.0_tip
- removed link link_8.0
- removed link link_9.0
- removed link palm
- removed link wrist
- added link index_L1, mass 0.00635888; visual mesh filename=models/idx-F1.STL
- added link index_L2, mass 0.00645; visual mesh filename=models/idx-F2.STL
- added link index_anchor
- added link middle_L1, mass 0.00635888; visual mesh filename=models/idx-F1.STL
- added link middle_L2, mass 0.00645; visual mesh filename=models/idx-F2.STL
- added link middle_anchor
- added link pinky_L1, mass 0.00635888; visual mesh filename=models/idx-F1.STL
- added link pinky_L2, mass 0.00645; visual mesh filename=models/idx-F2.STL
- added link pinky_anchor
- added link ring_L1, mass 0.00635888; visual mesh filename=models/idx-F1.STL
- added link ring_L2, mass 0.00645; visual mesh filename=models/idx-F2.STL
- added link ring_anchor
- added link thumb_L1, mass 0.00268342; visual mesh filename=models/thumb-F1.STL
- added link thumb_L2, mass 0.0055; visual mesh filename=models/thumb-F2.STL
- added link thumb_anchor
- added link thumb_base, mass 0.400; visual mesh filename=models/FB_palm_ref.STL
- link base_link: mass 0.4154 -> 0.200; geometry visual mesh filename=models/wristmesh.STL
Joints:
- removed joint joint_0.0
- removed joint joint_1.0
- removed joint joint_10.0
- removed joint joint_11.0
- removed joint joint_11.0_tip
- removed joint joint_12.0
- removed joint joint_13.0
- removed joint joint_14.0
- removed joint joint_15.0
- removed joint joint_15.0_tip
- removed joint joint_2.0
- removed joint joint_3.0
- removed joint joint_3.0_tip
- removed joint joint_4.0
- removed joint joint_5.0
- removed joint joint_6.0
- removed joint joint_7.0
- removed joint joint_7.0_tip
- removed joint joint_8.0
- removed joint joint_9.0
- removed joint palm_joint
- removed joint wrist_joint
- added joint idx_anchor: type fixed, parent index_L2, child index_anchor, origin xyz=31.5541e-3  -10.44e-3 0.14e-3 rpy=0 0 0
- added joint index_q1: type revolute, parent thumb_base, child index_L1, origin xyz=-9.49e-3 -13.04e-3 -62.95e-3 rpy=-1.982050 1.284473 -2.090591, axis 0 0 1, limit lower=0 upper=2.0943951 effort=6.0 velocity=8.0677777442
- added joint index_q2: type revolute, parent index_L1, child index_L2, origin xyz=38.472723e-3 3.257695e-3 0.000000e-3 rpy=0 0 0.084474, axis 0 0 1, limit lower=0.0 upper=2.6586 effort=6.0 velocity=8.0677777442
- added joint mid_anchor: type fixed, parent middle_L2, child middle_anchor, origin xyz=31.5541e-3  -10.44e-3 0.14e-3 rpy=0 0 0
- added joint middle_q1: type revolute, parent thumb_base, child middle_L1, origin xyz=9.653191e-3 -15.310271e-3 -67.853949e-3 rpy=-1.860531 1.308458 -1.896217, axis 0 0 1, limit lower=0 upper=2.0943951 effort=6.0 velocity=8.0677777442
- added joint middle_q2: type revolute, parent middle_L1, child middle_L2, origin xyz=38.472723e-3 3.257695e-3 0.000000 rpy=0 0 0.084474, axis 0 0 1, limit lower=0.0 upper=2.6586 effort=6.0 velocity=8.0677777442
- added joint pinky_q1: type revolute, parent thumb_base, child pinky_L1, origin xyz=49.521293e-3 -11.004583e-3 -63.029065e-3 rpy=-1.765110 1.322220 -1.658383, axis 0 0 1, limit lower=0 upper=2.0943951 effort=6.0 velocity=8.0677777442
- added joint pinky_q2: type revolute, parent pinky_L1, child pinky_L2, origin xyz=38.472723e-3 3.257695e-3 0.000000 rpy=0 0 0.084474, axis 0 0 1, limit lower=0.0 upper=2.6586 effort=6.0 velocity=8.0677777442
- added joint pnky_anchor: type fixed, parent pinky_L2, child pinky_anchor, origin xyz=31.5541e-3  -10.44e-3 0.14e-3 rpy=0 0 0
- added joint ring_q1: type revolute, parent thumb_base, child ring_L1, origin xyz=29.954260e-3 -14.212492e-3 -67.286105e-3 rpy=-1.716598 1.321452 -1.675862, axis 0 0 1, limit lower=0 upper=2.0943951 effort=6.0 velocity=8.0677777442
- added joint ring_q2: type revolute, parent ring_L1, child ring_L2, origin xyz=38.472723e-3 3.257695e-3 0.000000 rpy=0 0 0.084474, axis 0 0 1, limit lower=0.0 upper=2.6586 effort=6.0 velocity=8.0677777442
- added joint rng_anchor: type fixed, parent ring_L2, child ring_anchor, origin xyz=31.5541e-3  -10.44e-3 0.14e-3 rpy=0 0 0
- added joint thmb_anchor: type fixed, parent thumb_L2, child thumb_anchor, origin xyz=52.0012259e-3  28.0086971e-3 -.884835778e-3 rpy=0 0 0
- added joint thumb_q1: type revolute, parent thumb_base, child thumb_L1, origin xyz=0 0 0 rpy=0 0 3.330437, axis 0 0 1, limit lower=-2.0943951 upper=0 effort=1.2 velocity=40.338888721
- added joint thumb_q2: type revolute, parent thumb_L1, child thumb_L2, origin xyz=27.8283501e-3 0 -14.7507000e-3 rpy=4.450589592585541 0 0, axis 0 0 1, limit lower=0 upper=2.0943951 effort=6.0 velocity=8.0677777442
- added joint wrist2thumb: type fixed, parent base_link, child thumb_base, origin xyz=24.0476665e-3 3.78124745e-3 32.32964923e-3 rpy=3.14148426 0.08848813 3.14036612
- joint gripper_base_joint: origin xyz=0 0.045 0.045 rpy=0 -1.57 -1.57 -> xyz=0 0 0 rpy=0 0 3.14

File: assets/robot/xarm7_description/xarm7_ability_right.urdf (robot description, URDF)
Before this commit: robot xarm7, 32 links, 31 joints
Links:
- removed link link_0.0
- removed link link_1.0
- removed link link_10.0
- removed link link_11.0
- removed link link_11.0_tip
- removed link link_12.0
- removed link link_13.0
- removed link link_14.0
- removed link link_15.0
- removed link link_15.0_tip
- removed link link_2.0
- removed link link_3.0
- removed link link_3.0_tip
- removed link link_4.0
- removed link link_5.0
- removed link link_6.0
- removed link link_7.0
- removed link link_7.0_tip
- removed link link_8.0
- removed link link_9.0
- removed link palm
- removed link wrist
- added link index_L1, mass 0.00635888; visual mesh filename=models/idx-F1.STL
- added link index_L2, mass 0.00645; visual mesh filename=models/idx-F2.STL
- added link index_anchor
- added link middle_L1, mass 0.00635888; visual mesh filename=models/idx-F1.STL
- added link middle_L2, mass 0.00645; visual mesh filename=models/idx-F2.STL
- added link middle_anchor
- added link pinky_L1, mass 0.00635888; visual mesh filename=models/idx-F1.STL
- added link pinky_L2, mass 0.00645; visual mesh filename=models/idx-F2.STL
- added link pinky_anchor
- added link ring_L1, mass 0.00635888; visual mesh filename=models/idx-F1.STL
- added link ring_L2, mass 0.00645; visual mesh filename=models/idx-F2.STL
- added link ring_anchor
- added link thumb_L1, mass 0.00268342; visual mesh filename=models/thumb-F1-MIR.STL
- added link thumb_L2, mass 0.0055; visual mesh filename=models/thumb-F2.STL
- added link thumb_anchor
- added link thumb_base, mass 0.200; visual mesh filename=models/FB_palm_ref_MIR.STL
- link base_link: mass 0.4154 -> 0.200; geometry visual mesh filename=models/wristmesh.STL
Joints:
- removed joint joint_0.0
- removed joint joint_1.0
- removed joint joint_10.0
- removed joint joint_11.0
- removed joint joint_11.0_tip
- removed joint joint_12.0
- removed joint joint_13.0
- removed joint joint_14.0
- removed joint joint_15.0
- removed joint joint_15.0_tip
- removed joint joint_2.0
- removed joint joint_3.0
- removed joint joint_3.0_tip
- removed joint joint_4.0
- removed joint joint_5.0
- removed joint joint_6.0
- removed joint joint_7.0
- removed joint joint_7.0_tip
- removed joint joint_8.0
- removed joint joint_9.0
- removed joint palm_joint
- removed joint wrist_joint
- added joint idx_anchor: type fixed, parent index_L2, child index_anchor, origin xyz=31.5541e-3  -10.44e-3 0.14e-3 rpy=0 0 0
- added joint index_q1: type revolute, parent thumb_base, child index_L1, origin xyz= 9.49e-3 -13.04e-3 -62.95e-3  rpy= -1.1595426535897932 1.284473 -1.0510016535897932 , axis 0 0 1, limit lower=0 upper=2.0943951 effort=6.0 velocity=8.0677777442
- added joint index_q2: type revolute, parent index_L1, child index_L2, origin xyz=38.472723e-3 3.257695e-3 0.000000e-3 rpy=0 0 0.084474, axis 0 0 1, limit lower=0.0 upper=2.6586 effort=6.0 velocity=8.0677777442
- added joint mid_anchor: type fixed, parent middle_L2, child middle_anchor, origin xyz=31.5541e-3  -10.44e-3 0.14e-3 rpy=0 0 0
- added joint middle_q1: type revolute, parent thumb_base, child middle_L1, origin xyz= -9.653191e-3 -15.310271e-3 -67.853949e-3  rpy= -1.2810616535897934 1.308458 -1.2453756535897933 , axis 0 0 1, limit lower=0 upper=2.0943951 effort=6.0 velocity=8.0677777442
- added joint middle_q2: type revolute, parent middle_L1, child middle_L2, origin xyz=38.472723e-3 3.257695e-3 0.000000 rpy=0 0 0.084474, axis 0 0 1, limit lower=0.0 upper=2.6586 effort=6.0 velocity=8.0677777442
- added joint pinky_q1: type revolute, parent thumb_base, child pinky_L1, origin xyz= -49.521293e-3 -11.004583e-3 -63.029065e-3  rpy= -1.3764826535897934 1.32222 -1.4832096535897932 , axis 0 0 1, limit lower=0 upper=2.0943951 effort=6.0 velocity=8.0677777442
- added joint pinky_q2: type revolute, parent pinky_L1, child pinky_L2, origin xyz=38.472723e-3 3.257695e-3 0.000000 rpy=0 0 0.084474, axis 0 0 1, limit lower=0.0 upper=2.6586 effort=6.0 velocity=8.0677777442
- added joint pnky_anchor: type fixed, parent pinky_L2, child pinky_anchor, origin xyz=31.5541e-3  -10.44e-3 0.14e-3 rpy=0 0 0
- added joint ring_q1: type revolute, parent thumb_base, child ring_L1, origin xyz= -29.95426e-3 -14.212492e-3 -67.286105e-3  rpy= -1.424994653589793 1.321452 -1.4657306535897934 , axis 0 0 1, limit lower=0 upper=2.0943951 effort=6.0 velocity=8.0677777442
- added joint ring_q2: type revolute, parent ring_L1, child ring_L2, origin xyz=38.472723e-3 3.257695e-3 0.000000 rpy=0 0 0.084474, axis 0 0 1, limit lower=0.0 upper=2.6586 effort=6.0 velocity=8.0677777442
- added joint rng_anchor: type fixed, parent ring_L2, child ring_anchor, origin xyz=31.5541e-3  -10.44e-3 0.14e-3 rpy=0 0 0
- added joint thmb_anchor: type fixed, parent thumb_L2, child thumb_anchor, origin xyz=52.00122724e-3 28.00869333e-3 6.98483578e-3 rpy=0 0 0
- added joint thumb_q1: type revolute, parent thumb_base, child thumb_L1, origin xyz= 0.0 0.0 0.0  rpy= 3.141592653589793 -0.0 -0.18884434641020664 , axis 0 0 1, limit lower=-2.0943951 upper=0 effort=1.2 velocity=40.338888721
- added joint thumb_q2: type revolute, parent thumb_L1, child thumb_L2, origin xyz= 27.8283501e-3 1.7436510745838653e-19 14.7507e-3  rpy= 1.832595714594045 -0.0 5.366520605522463e-18 , axis 0 0 1, limit lower=0 upper=2.0943951 effort=6.0 velocity=8.0677777442
- added joint wrist2thumb: type fixed, parent base_link, child thumb_base, origin xyz=-24.0476665e-3 3.78124745e-3 32.32964923e-3 rpy=3.14148426 -0.08848813 -3.14036612
- joint gripper_base_joint: origin xyz=0 0.045 0.045 rpy=0 -1.57 -1.57 -> xyz=0 0 0 rpy=0 0 3.14
